File: sublink/_autosave-sublink.kicad_sch (KiCad schematic)
At the start: 45 parts, among them J1 ZL315-4SGH, Q1 Q_PMOS_GSD, SW1 SW_Push, SW2 SW_Push, SW3 SW_Push, U1 ATtiny414-SS, U2 OKY3402, U3 JS202011

Commit message: finishing touches, silkscreen etc
Changed lines of the file:
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@@
   (junction (at 96.52 74.93) (diameter 0) (color 0 0 0 0)
-  )
-  (bus_entry (at 179.705 51.435) (size 2.54 2.54)
-    (stroke (width 0) (type default) (color 0 0 0 0))
   )
   (wire (pts (xy 177.8 60.96) (xy 177.8 64.77))
