File: sublink/sublink.kicad_pcb (KiCad board)
At the start: 2 copper layers, 94.8 x 82.1 mm, 45 parts, among them J1 ZL315-4SGH, Q1 Q_PMOS_GSD, SW1 SW_Push, SW2 SW_Push, SW3 SW_Push, U1 ATtiny414-SS, U2 OKY3402, U3 JS202011

Commit message: dot routing
Parts:
- turned D2 to -40 degrees
Routing:
- net GND: track 9.39 -> 13.7 mm, vias 0 -> 3
- net Net-(D2-Pad2): track 0.00 -> 1.58 mm, vias 0 -> 1
- net Net-(D1-Pad2): track 0.00 -> 1.45 mm, vias 0 -> 1
- net Net-(D3-Pad2): track 0.00 -> 1.34 mm, vias 0 -> 1
Changed lines of the file:
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@@
   )
   (footprint "LED_SMD:LED_0805_2012Metric_Pad1.15x1.40mm_HandSolder" (layer "F.Cu")
-    (at 198.40815 115.045656 -25)
+    (at 198.40815 115.045656 -40)
     (descr "LED SMD 0805 (2012 Metric), square (rectangular) end terminal, IPC_7351 nominal, (Body size source: https://docs.google.com/spreadsheets/d/1BsfQQcO9C6DZCsRaXUlFlo91Tg2WpOkGARC1WS5S8t0/edit?usp=sharing), generated with kicad-footprint-generator")
     (tags "LED handsolder")
@@
     (property "Sheetname" "")
     (attr smd)
-    (fp_text reference "D2" (at 0 -1.65 155) (layer "F.SilkS")
+    (fp_text reference "D2" (at 0 -1.65 140) (layer "F.SilkS")
       (effects (font (size 1 1) (thickness 0.15)))
     )
-    (fp_text value "LED" (at 0 1.65 155) (layer "F.Fab")
+    (fp_text value "LED" (at 0 1.65 140) (layer "F.Fab")
       (effects (font (size 1 1) (thickness 0.15)))
     )
-    (fp_text user "${REFERENCE}" (at 0 0 155) (layer "F.Fab")
+    (fp_text user "${REFERENCE}" (at 0 0 140) (layer "F.Fab")
       (effects (font (size 0.5 0.5) (thickness 0.08)))
     )
@@
     (fp_line (start -1 -0.3) (end -1 0.6) (layer "F.Fab") (width 0.1))
     (fp_line (start -1 0.6) (end 1 0.6) (layer "F.Fab") (width 0.1))
-    (pad "1" smd roundrect (at -1.025 0 335) (size 1.15 1.4) (layers "F.Cu" "F.Paste" "F.Mask") (roundrect_rratio 0.217391)
+    (pad "1" smd roundrect (at -1.025 0 320) (size 1.15 1.4) (layers "F.Cu" "F.Paste" "F.Mask") (roundrect_rratio 0.217391)
       (net 6 "GND") (pinfunction "K") (pintype "passive"))
-    (pad "2" smd roundrect (at 1.025 0 335) (size 1.15 1.4) (layers "F.Cu" "F.Paste" "F.Mask") (roundrect_rratio 0.217391)
+    (pad "2" smd roundrect (at 1.025 0 320) (size 1.15 1.4) (layers "F.Cu" "F.Paste" "F.Mask") (roundrect_rratio 0.217391)
       (net 8 "Net-(D2-Pad2)") (pinfunction "A") (pintype "passive"))
     (model "${KICAD6_3DMODEL_DIR}/LED_SMD.3dshapes/LED_0805_2012Metric.wrl"
@@
   (segment (start 162.052 105.918) (end 155.194 105.918) (width 0.3) (layer "B.Cu") (net 5))
   (segment (start 169.488434 99.878032) (end 169.223828 100.142638) (width 0.3) (layer "B.Cu") (net 5))
+  (segment (start 174.214844 71.308909) (end 174.214844 72.868844) (width 0.25) (layer "F.Cu") (net 6))
+  (segment (start 148.781577 113.092423) (end 149.606 112.268) (width 0.25) (layer "F.Cu") (net 6))
+  (segment (start 174.214844 72.868844) (end 174.244 72.898) (width 0.25) (layer "F.Cu") (net 6))
+  (segment (start 197.622954 114.386799) (end 197.444799 114.386799) (width 0.25) (layer "F.Cu") (net 6))
+  (segment (start 148.587965 113.092423) (end 148.781577 113.092423) (width 0.25) (layer "F.Cu") (net 6))
+  (segment (start 197.444799 114.386799) (end 196.596 113.538) (width 0.25) (layer "F.Cu") (net 6))
+  (via (at 196.596 113.538) (size 0.8) (drill 0.4) (layers "F.Cu" "B.Cu") (net 6))
+  (via (at 174.244 72.898) (size 0.8) (drill 0.4) (layers "F.Cu" "B.Cu") (net 6))
+  (via (at 149.606 112.268) (size 0.8) (drill 0.4) (layers "F.Cu" "B.Cu") (net 6))
   (segment (start 183.350002 122.372002) (end 185.05 124.072) (width 0.3) (layer "B.Cu") (net 6))
   (segment (start 160.4415 93.7045) (end 157.226 90.489) (width 0.9) (layer "B.Cu") (net 6))
   (segment (start 181 122.372002) (end 183.350002 122.372002) (width 0.3) (layer "B.Cu") (net 6))
   (segment (start 160.528 93.7045) (end 160.4415 93.7045) (width 0.9) (layer "B.Cu") (net 6))
+  (segment (start 174.214844 67.847156) (end 174.244 67.818) (width 0.25) (layer "F.Cu") (net 7))
+  (segment (start 174.214844 69.258909) (end 174.214844 67.847156) (width 0.25) (layer "F.Cu") (net 7))
+  (via (at 174.244 67.818) (size 0.8) (drill 0.4) (layers "F.Cu" "B.Cu") (net 7))
+  (segment (start 199.193346 115.704513) (end 199.524513 115.704513) (width 0.25) (layer "F.Cu") (net 8))
+  (segment (start 199.524513 115.704513) (end 200.406 116.586) (width 0.25) (layer "F.Cu") (net 8))
+  (via (at 200.406 116.586) (size 0.8) (drill 0.4) (layers "F.Cu" "B.Cu") (net 8))
+  (segment (start 146.955863 114.410137) (end 146.05 115.316) (width 0.25) (layer "F.Cu") (net 9))
+  (segment (start 147.017573 114.410137) (end 146.955863 114.410137) (width 0.25) (layer "F.Cu") (net 9))
+  (via (at 146.05 115.316) (size 0.8) (drill 0.4) (layers "F.Cu" "B.Cu") (net 9))
   (segment (start 184.45 107.472) (end 185.05 108.072) (width 0.9) (layer "B.Cu") (net 10))
   (segment (start 197.8375 103.272) (end 196.3375 101.772) (width 0.9) (layer "B.Cu") (net 10))

Commit message: finishing touches, silkscreen etc
Parts:
- moved U2 37.3 mm to (195.0, 115.4), turned to 90 degrees
- moved R1 20.0 mm to (154.0, 84.5), turned to 45 degrees
- moved R9 19.8 mm to (189.8, 103.7), turned to 0 degrees
- moved BT1 3.73 mm to (180.2, 103.7)
- moved R2 1.84 mm to (144.6, 102.6)
- moved H2 0.64 mm to (214.4, 123.5)
- moved H1 0.28 mm to (173.2, 51.9)
- moved H3 0.24 mm to (131.8, 123.4)
Connections:
- D2 pad 2: Net-(D2-Pad2) -> Net-(R3-Pad2)
- D3 pad 2: Net-(D3-Pad2) -> Net-(R2-Pad2)
- J1 pad 1: Net-(J1-Pad1) -> Net-(U3-Pad1)
- R2 pad 2: Net-(D2-Pad2) -> Net-(R2-Pad2)
- R3 pad 2: Net-(D3-Pad2) -> Net-(R3-Pad2)
- U3 pad 1: unconnected-(U3-Pad1) -> Net-(U3-Pad1)
- U3 pad 3: Net-(J1-Pad1) -> unconnected-(U3-Pad3)
Routing:
- net Net-(R3-Pad2): track 0.00 -> 59.5 mm, vias 0 -> 1
- net unconnected-(U3-Pad1): track 35.3 -> 0.00 mm
- net Net-(U3-Pad1): track 0.00 -> 35.3 mm
- net Net-(D1-Pad2): track 1.45 -> 31.0 mm
- net Net-(D23-Pad2): track 42.2 -> 18.2 mm
- net Net-(R2-Pad2): track 0.00 -> 13.7 mm, vias 0 -> 1
- net GND: track 13.7 -> 25.4 mm, vias 3 -> 19
- net Net-(R1-Pad1): track 13.4 -> 6.24 mm
- net Net-(D2-Pad2): track 1.58 -> 0.00 mm, vias 1 -> 0
- net Net-(D3-Pad2): track 1.34 -> 0.00 mm, vias 1 -> 0
- net Net-(BT1-Pad1): track 22.2 -> 23.2 mm
- net Net-(R3-Pad1): track 6.90 -> 7.62 mm
- net Net-(R2-Pad1): track 14.0 -> 13.3 mm
- net VCC: vias 0 -> 1
- net Net-(D22-Pad1): vias 0 -> 1
- added copper zone on F.Cu, net (none)
- added copper zone on B.Cu, net GND
- added copper zone on F.Cu, net GND
Other:
- board text added: "5V"
- board text added: "ATTINY414"
- board text added: "GND"
- board text added: "JLCJLCJLCJLC"
- board text added: "NC"
- board text added: "OFF/PRG"
- board text added: "ON"
- board text added: "UPDI"
- board text added: "github.com/ ptrbroz/SU_blink"
